File: ThumbsUp.kicad_pcb (KiCad board)
At the start: 2 copper layers, 247.3 x 91.5 mm, 150 parts, among them IC1 RP2040, IC2 W25Q128JVSIM, IC3 RP2040, IC4 W25Q128JVSIM, J1 Conn_01x04_Male, J10 Raiser_Male, J11 Raiser_Female, J12 Raiser_Male, J13 Raiser_Female, J14 Raiser_Male, J15 Raiser_Female, J16 Raiser_Male, J17 Raiser_Female, J18 Raiser_Male, J19 Raiser_Female, J2 Conn_01x04_Male, J20 Conn_01x04_Female, J21 Conn_01x04_Female, J22 Conn_01x04_Female, J23 Conn_01x04_Female, J24 Conn_01x04_Male, J25 Conn_01x04_Male, J26 Conn_01x04_Male, J27 Conn_01x04_Male, J28 Conn_01x04_Female, J29 Conn_01x04_Female, J3 Conn_01x04_Female, J30 Conn_01x04_Female, J31 Conn_01x04_Female, J32 USB_C_Receptacle_USB2.0, J33 Raiser_Male, J34 Raiser_Female, J35 Raiser_Male, J36 STX-3501-3N, J37 USB_C_Receptacle_USB2.0, J38 Raiser_Female, J39 Raiser_Male, J4 Conn_01x04_Male, J40 Raiser_Female, J41 Raiser_Male, J42 Raiser_Female, J43 Raiser_Male, J44 Raiser_Female, J45 Raiser_Male, J46 STX-3501-3N, J5 Conn_01x04_Female, J6 Conn_01x04_Male, J7 Conn_01x04_Male, J8 Conn_01x04_Male, J9 Raiser_Female, U1 NCP1117-3.3_SOT223, U2 NCP1117-3.3_SOT223, Y1 ABLS-12.000MHZ-B4-T, Y2 ABLS-12.000MHZ-B4-T

Commit message: Rearranged the header pins to match the actual positions.
Parts:
- added J47: Raiser_Female, Connector_PinSocket_2.54mm:PinSocket_1x04_P2.54mm_Vertical, F.Cu at (154.4, 464.5)
- added J48: Raiser_Male, Connector_PinHeader_2.54mm:PinHeader_1x04_P2.54mm_Vertical, B.Cu at (156.9, 342.0)
- J1, J10, J12, J14, J16, J18, J2, J24, J25, J26, J27, J33, J35, J4, J6, J7, J8: moved to B.Cu
- J17, J19, J34, J9: moved to F.Cu
- moved BOOTSEL2 309.9 mm to (280.2, 478.6)
- moved C18 309.9 mm to (294.6, 490.6)
- moved C19 309.9 mm to (286.5, 480.1)
- moved C20 309.9 mm to (290.2, 486.5)
- moved C21 309.9 mm to (277.9, 473.5)
- moved C22 309.9 mm to (253.1, 487.2)
- moved C23 309.9 mm to (290.2, 489.4)
- moved C24 309.9 mm to (269.8, 472.3)
- moved C25 309.9 mm to (292.5, 496.5)
- moved C26 309.9 mm to (294.6, 487.6)
- moved C27 309.9 mm to (292.5, 499.4)
- moved C28 309.9 mm to (252.5, 473.3)
- moved C29 309.9 mm to (251.3, 470.4)
- moved C30 309.9 mm to (246.9, 470.0)
- moved C31 309.9 mm to (242.5, 470.0)
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Connections:
- BOOTSEL1 pad 3: GND -> L-BASE
- BOOTSEL1 pad 4: GND -> L-BASE
- BOOTSEL2 pad 3: GND -> L-BASE
- BOOTSEL2 pad 4: GND -> L-BASE
- C1 pad 1: +3V3 -> L-RING1
- C1 pad 2: GND -> L-BASE
- C10 pad 1: +3V3 -> L-RING1
- C10 pad 2: GND -> L-BASE
- C11 pad 1: +3V3 -> L-RING1
- C11 pad 2: GND -> L-BASE
- C12 pad 2: GND -> L-BASE
- C13 pad 2: GND -> L-BASE
- C14 pad 2: GND -> L-BASE
- C15 pad 1: +3V3 -> L-RING1
- C15 pad 2: GND -> L-BASE
- C16 pad 1: +3V3 -> L-RING1
- C16 pad 2: GND -> L-BASE
- C17 pad 1: +3V3 -> L-RING1
- C17 pad 2: GND -> L-BASE
- C18 pad 1: +3V3 -> L-RING1
- C18 pad 2: GND -> L-BASE
- C19 pad 1: +3V3 -> L-RING1
- C19 pad 2: GND -> L-BASE
- C2 pad 1: +3V3 -> L-RING1
- C2 pad 2: GND -> L-BASE
- C20 pad 1: +3V3 -> L-RING1
- C20 pad 2: GND -> L-BASE
- C21 pad 2: GND -> L-BASE
- C22 pad 2: GND -> L-BASE
- C23 pad 1: +3V3 -> L-RING1
- C23 pad 2: GND -> L-BASE
- C24 pad 2: GND -> L-BASE
- C25 pad 1: +3V3 -> L-RING1
- C25 pad 2: GND -> L-BASE
- C26 pad 2: GND -> L-BASE
- C27 pad 1: +3V3 -> L-RING1
- C27 pad 2: GND -> L-BASE
- C28 pad 2: GND -> L-BASE
- C29 pad 1: +3V3 -> L-RING1
- C29 pad 2: GND -> L-BASE
- C3 pad 1: +3V3 -> L-RING1
- C3 pad 2: GND -> L-BASE
- C30 pad 1: +3V3 -> L-RING1
- C30 pad 2: GND -> L-BASE
- C31 pad 1: +3V3 -> L-RING1
- C31 pad 2: GND -> L-BASE
- C32 pad 1: +3V3 -> L-RING1
- C32 pad 2: GND -> L-BASE
- C4 pad 2: GND -> L-BASE
- C5 pad 2: GND -> L-BASE
- C6 pad 1: +3V3 -> L-RING1
- C6 pad 2: GND -> L-BASE
- C7 pad 1: +3V3 -> L-RING1
- C7 pad 2: GND -> L-BASE
- C8 pad 2: GND -> L-BASE
- C9 pad 2: GND -> L-BASE
- IC1 pad 1: +3V3 -> L-RING1
- IC1 pad 10: +3V3 -> L-RING1
- IC1 pad 19: GND -> L-BASE
- IC1 pad 22: +3V3 -> L-RING1
- IC1 pad 26: GND -> L-BASE
- IC1 pad 32: Net-(IC1-Pad32) -> L-TIP
- IC1 pad 33: +3V3 -> L-RING1
- IC1 pad 42: +3V3 -> L-RING1
- IC1 pad 43: +3V3 -> L-RING1
- IC1 pad 44: +3V3 -> L-RING1
- IC1 pad 48: +3V3 -> L-RING1
- IC1 pad 49: +3V3 -> L-RING1
- IC1 pad 57: GND -> L-BASE
- IC2 pad 4: GND -> L-BASE
- IC2 pad 8: +3V3 -> L-RING1
- IC3 pad 1: +3V3 -> L-RING1
- IC3 pad 10: +3V3 -> L-RING1
- IC3 pad 19: GND -> L-BASE
- IC3 pad 22: +3V3 -> L-RING1
- IC3 pad 26: GND -> L-BASE
- IC3 pad 32: Net-(IC3-Pad32) -> R-TIP
- IC3 pad 33: +3V3 -> L-RING1
- IC3 pad 42: +3V3 -> L-RING1
- IC3 pad 43: +3V3 -> L-RING1
- IC3 pad 44: +3V3 -> L-RING1
- IC3 pad 48: +3V3 -> L-RING1
- IC3 pad 49: +3V3 -> L-RING1
- IC3 pad 57: GND -> L-BASE
- IC4 pad 4: GND -> L-BASE
- IC4 pad 8: +3V3 -> L-RING1
- J20 pad 4: GND -> L-BASE
- J24 pad 4: GND -> L-BASE
- J32 pad A1: GND -> L-BASE
- J32 pad A12: GND -> L-BASE
- J32 pad B1: GND -> L-BASE
- J32 pad B12: GND -> L-BASE
- J32 pad S1: GND -> L-BASE
- J36 pad 1: Net-(J36-Pad1) -> L-BASE
- J36 pad 2: Net-(J36-Pad2) -> L-TIP
- J36 pad 3: Net-(J36-Pad3) -> L-RING1
- J37 pad A1: GND -> L-BASE
- J37 pad A12: GND -> L-BASE
- J37 pad B1: GND -> L-BASE
- J37 pad B12: GND -> L-BASE
- J37 pad S1: GND -> L-BASE
- J4 pad 1: GND -> L-BASE
- J46 pad 1: Net-(J46-Pad1) -> L-BASE
- J46 pad 2: Net-(J46-Pad2) -> R-TIP
- J46 pad 3: Net-(J46-Pad3) -> L-RING1
- J6 pad 1: GND -> L-BASE
- MX10 pad 1: GND -> L-BASE
- MX14 pad 1: GND -> L-BASE
- MX15 pad 1: GND -> L-BASE
- MX16 pad 1: GND -> L-BASE
- MX17 pad 1: GND -> L-BASE
- MX19 pad 1: GND -> L-BASE
- MX20 pad 1: GND -> L-BASE
- MX21 pad 1: GND -> L-BASE
- MX23 pad 1: GND -> L-BASE
- MX24 pad 1: GND -> L-BASE
- MX25 pad 1: GND -> L-BASE
- MX27 pad 1: GND -> L-BASE
- MX28 pad 1: GND -> L-BASE
- MX29 pad 1: GND -> L-BASE
- MX34 pad 1: GND -> L-BASE
- MX38 pad 1: GND -> L-BASE
- R10 pad 2: GND -> L-BASE
- R11 pad 1: GND -> L-BASE
- R13 pad 2: +3V3 -> L-RING1
- R7 pad 2: +3V3 -> L-RING1
- R8 pad 2: GND -> L-BASE
- R9 pad 1: GND -> L-BASE
- RUN1 pad 3: GND -> L-BASE
- RUN1 pad 4: GND -> L-BASE
- RUN2 pad 3: GND -> L-BASE
- RUN2 pad 4: GND -> L-BASE
- U1 pad 1: GND -> L-BASE
- U1 pad 2: +3V3 -> L-RING1
- U2 pad 1: GND -> L-BASE
- U2 pad 2: +3V3 -> L-RING1
Other:
- board size 247.3 x 91.5 mm -> 247.3 x 275.2 mm

Commit message: Traced the top  and bottom plates.
Parts:
- moved J48 5.70 mm to (156.8, 336.3), turned to 180 degrees
- moved J14 5.70 mm to (132.5, 336.4), turned to 180 degrees
- moved J10 4.46 mm to (93.8, 339.9), turned to 180 degrees
- moved J33 4.45 mm to (195.6, 339.7), turned to 180 degrees
- moved J35 4.16 mm to (169.4, 325.8), turned to 75 degrees
- moved J18 4.15 mm to (119.9, 325.9), turned to 285 degrees
- moved J6 3.87 mm to (190.6, 347.4), turned to 90 degrees
- moved J4 3.82 mm to (99.0, 347.6), turned to 270 degrees
- moved MX18 2.77 mm to (121.3, 337.8), turned to 0 degrees
- moved MX30 2.72 mm to (168.2, 337.7), turned to 180 degrees
- moved MX26 2.14 mm to (186.7, 337.7), turned to 180 degrees
- moved MX22 2.10 mm to (102.8, 337.8), turned to 0 degrees
Connections:
- J1 pad 1: Net-(J1-Pad1) -> L-BASE
- J2 pad 1: Net-(J2-Pad1) -> K_ESC
- J2 pad 2: Net-(J2-Pad2) -> K_Q
- J2 pad 3: Net-(J2-Pad3) -> K_W
- J2 pad 4: Net-(J2-Pad4) -> K_E
- J20 pad 4: L-BASE -> Net-(J20-Pad4)
- J21 pad 1: K_ESC -> Net-(J21-Pad1)
- J21 pad 2: K_Q -> Net-(J21-Pad2)
- J21 pad 3: K_W -> Net-(J21-Pad3)
- J21 pad 4: K_E -> Net-(J21-Pad4)
- J22 pad 1: K_TAB -> Net-(J22-Pad1)
- J22 pad 2: K_A -> Net-(J22-Pad2)
- J22 pad 3: K_S -> Net-(J22-Pad3)
- J22 pad 4: K_D -> Net-(J22-Pad4)
- J23 pad 1: K_LCTL -> Net-(J23-Pad1)
- J23 pad 2: K_Z -> Net-(J23-Pad2)
- J23 pad 3: K_X -> Net-(J23-Pad3)
- J23 pad 4: K_C -> Net-(J23-Pad4)
- J24 pad 1: Net-(J24-Pad1) -> L-BASE
- J24 pad 4: L-BASE -> Net-(J24-Pad4)
- J26 pad 1: K_ENT -> K_K
- J26 pad 2: K_SEMICOL -> K_L
- J26 pad 3: K_L -> K_SEMICOL
- J26 pad 4: K_K -> K_ENT
- J27 pad 1: K_RCTL -> K_COMM
- J27 pad 2: K_SLASH -> K_DOT
- J27 pad 3: K_DOT -> K_SLASH
- J27 pad 4: K_COMM -> K_RCTL
- J3 pad 1: Net-(J3-Pad1) -> L-BASE
- J3 pad 2: Net-(J3-Pad2) -> K_LSFT
- J3 pad 4: Net-(J3-Pad4) -> K_RSE
- J4 pad 1: L-BASE -> Net-(J4-Pad1)
- J4 pad 2: K_LSFT -> Net-(J4-Pad2)
- J4 pad 4: K_RSE -> Net-(J4-Pad4)
- J5 pad 2: Net-(J5-Pad2) -> K_LWR
- J5 pad 3: Net-(J5-Pad3) -> K_RSFT
- J5 pad 4: Net-(J5-Pad4) -> L-BASE
- J6 pad 1: L-BASE -> Net-(J6-Pad1)
- J6 pad 2: K_LWR -> Net-(J6-Pad2)
- J6 pad 4: K_RSFT -> Net-(J6-Pad4)
- J7 pad 1: Net-(J7-Pad1) -> K_TAB
- J7 pad 2: Net-(J7-Pad2) -> K_A
- J7 pad 3: Net-(J7-Pad3) -> K_S
- J7 pad 4: Net-(J7-Pad4) -> K_D
- J8 pad 1: Net-(J8-Pad1) -> K_LCTL
- J8 pad 2: Net-(J8-Pad2) -> K_Z
- J8 pad 3: Net-(J8-Pad3) -> K_X
- J8 pad 4: Net-(J8-Pad4) -> K_C
- MX1 pad 1: Net-(J1-Pad4) -> Net-(J20-Pad1)
- MX1 pad 2: Net-(J2-Pad1) -> Net-(J21-Pad1)
- MX11 pad 1: Net-(J1-Pad4) -> Net-(J20-Pad1)
- MX11 pad 2: Net-(J2-Pad4) -> Net-(J21-Pad4)
- MX12 pad 1: Net-(J1-Pad4) -> Net-(J20-Pad1)
- MX12 pad 2: Net-(J7-Pad4) -> Net-(J22-Pad4)
- MX13 pad 1: Net-(J1-Pad4) -> Net-(J20-Pad1)
- MX13 pad 2: Net-(J8-Pad4) -> Net-(J23-Pad4)
- MX18 pad 1: Net-(J3-Pad1) -> Net-(J4-Pad1)
- MX18 pad 2: Net-(J3-Pad4) -> Net-(J4-Pad4)
- MX2 pad 1: Net-(J1-Pad4) -> Net-(J20-Pad1)
- MX2 pad 2: Net-(J7-Pad1) -> Net-(J22-Pad1)
- MX22 pad 1: Net-(J3-Pad1) -> Net-(J4-Pad1)
- MX22 pad 2: Net-(J3-Pad2) -> Net-(J4-Pad2)
- MX26 pad 1: Net-(J5-Pad1) -> Net-(J6-Pad4)
- MX26 pad 2: Net-(J5-Pad4) -> Net-(J6-Pad3)
- MX3 pad 1: Net-(J1-Pad4) -> Net-(J20-Pad1)
- MX3 pad 2: Net-(J8-Pad1) -> Net-(J23-Pad1)
- MX30 pad 1: Net-(J5-Pad1) -> Net-(J6-Pad4)
- MX30 pad 2: Net-(J5-Pad2) -> Net-(J6-Pad2)
- MX31 pad 1: Net-(J28-Pad4) -> Net-(J28-Pad1)
- MX32 pad 1: Net-(J28-Pad4) -> Net-(J28-Pad1)
- MX32 pad 2: Net-(J30-Pad4) -> Net-(J30-Pad1)
- MX33 pad 1: Net-(J28-Pad4) -> Net-(J28-Pad1)
- MX33 pad 2: Net-(J31-Pad4) -> Net-(J31-Pad1)
- MX35 pad 1: Net-(J28-Pad4) -> Net-(J28-Pad1)
- MX36 pad 1: Net-(J28-Pad4) -> Net-(J28-Pad1)
- MX36 pad 2: Net-(J30-Pad3) -> Net-(J30-Pad2)
- MX37 pad 1: Net-(J28-Pad4) -> Net-(J28-Pad1)
- MX37 pad 2: Net-(J31-Pad3) -> Net-(J31-Pad2)
- MX39 pad 1: Net-(J28-Pad4) -> Net-(J28-Pad1)
- MX4 pad 1: Net-(J1-Pad4) -> Net-(J20-Pad1)
- MX4 pad 2: Net-(J2-Pad2) -> Net-(J21-Pad2)
- MX40 pad 1: Net-(J28-Pad4) -> Net-(J28-Pad1)
- MX40 pad 2: Net-(J30-Pad2) -> Net-(J30-Pad3)
- MX41 pad 1: Net-(J28-Pad4) -> Net-(J28-Pad1)
- MX41 pad 2: Net-(J31-Pad2) -> Net-(J31-Pad3)
- MX42 pad 1: Net-(J28-Pad4) -> Net-(J28-Pad1)
- MX43 pad 1: Net-(J28-Pad4) -> Net-(J28-Pad1)
- MX43 pad 2: Net-(J30-Pad1) -> Net-(J30-Pad4)
- MX44 pad 1: Net-(J28-Pad4) -> Net-(J28-Pad1)
- MX44 pad 2: Net-(J31-Pad1) -> Net-(J31-Pad4)
- MX5 pad 1: Net-(J1-Pad4) -> Net-(J20-Pad1)
- MX5 pad 2: Net-(J7-Pad2) -> Net-(J22-Pad2)
- MX6 pad 1: Net-(J1-Pad4) -> Net-(J20-Pad1)
- MX6 pad 2: Net-(J8-Pad2) -> Net-(J23-Pad2)
- MX7 pad 1: Net-(J1-Pad4) -> Net-(J20-Pad1)
- MX7 pad 2: Net-(J2-Pad3) -> Net-(J21-Pad3)
- MX8 pad 1: Net-(J1-Pad4) -> Net-(J20-Pad1)
- MX8 pad 2: Net-(J7-Pad3) -> Net-(J22-Pad3)
- MX9 pad 1: Net-(J1-Pad4) -> Net-(J20-Pad1)
- MX9 pad 2: Net-(J8-Pad3) -> Net-(J23-Pad3)
Routing:
- net Net-(J28-Pad1): track 0.00 -> 323.3 mm
- net Net-(J20-Pad1): track 0.00 -> 291.0 mm
- net Net-(J23-Pad1): track 0.00 -> 85.0 mm
- net Net-(J29-Pad1): track 0.00 -> 85.0 mm
- net Net-(J21-Pad1): track 0.00 -> 84.3 mm
- net Net-(J22-Pad1): track 0.00 -> 84.2 mm
- net Net-(J30-Pad4): track 0.00 -> 83.7 mm
- net Net-(J31-Pad4): track 0.00 -> 83.4 mm
- net Net-(J29-Pad2): track 0.00 -> 55.4 mm
- net Net-(J31-Pad3): track 0.00 -> 54.5 mm
- net Net-(J30-Pad3): track 0.00 -> 54.3 mm
- net Net-(J22-Pad2): track 0.00 -> 53.3 mm
- net Net-(J23-Pad2): track 0.00 -> 53.3 mm
- net Net-(J6-Pad2): track 0.00 -> 53.0 mm
- net Net-(J21-Pad2): track 0.00 -> 52.9 mm
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Other:
- board size 247.3 x 275.2 mm -> 247.3 x 280.2 mm

Commit message: Retracing the plates.
Parts:
- moved IC2 119.7 mm to (122.2, 462.0), turned to 90 degrees
- moved U1 98.9 mm to (110.6, 444.1), turned to 270 degrees
- moved Y1 93.5 mm to (96.0, 455.9), turned to 270 degrees
- moved IC1 2.30 mm to (109.8, 457.4), turned to 90 degrees
- turned MX21 to 0 degrees
Connections:
- J1 pad 1: L-BASE -> Net-(J1-Pad1)
- J16 pad 1: Net-(J16-Pad1) -> K_TAB
- J16 pad 2: Net-(J16-Pad2) -> K_A
- J16 pad 3: Net-(J16-Pad3) -> K_S
- J16 pad 4: Net-(J16-Pad4) -> K_D
- J2 pad 1: K_ESC -> Net-(J2-Pad1)
- J2 pad 2: K_Q -> Net-(J2-Pad2)
- J2 pad 3: K_W -> Net-(J2-Pad3)
- J2 pad 4: K_E -> L-BASE
- J45 pad 1: Net-(J45-Pad1) -> K_ESC
- J45 pad 2: Net-(J45-Pad2) -> K_Q
- J45 pad 3: Net-(J45-Pad3) -> K_W
- J45 pad 4: Net-(J45-Pad4) -> K_E
- J7 pad 1: K_TAB -> Net-(J7-Pad1)
- J7 pad 2: K_A -> Net-(J7-Pad2)
- J7 pad 3: K_S -> Net-(J7-Pad3)
- J7 pad 4: K_D -> Net-(J7-Pad4)
- MX1 pad 1: Net-(J20-Pad1) -> Net-(J21-Pad4)
- MX1 pad 2: Net-(J21-Pad1) -> Net-(J44-Pad1)
- MX11 pad 1: Net-(J20-Pad1) -> Net-(J21-Pad4)
- MX11 pad 2: Net-(J21-Pad4) -> Net-(J44-Pad4)
- MX12 pad 1: Net-(J20-Pad1) -> Net-(J21-Pad4)
- MX12 pad 2: Net-(J22-Pad4) -> Net-(J15-Pad4)
- MX13 pad 1: Net-(J20-Pad1) -> Net-(J21-Pad4)
- MX2 pad 1: Net-(J20-Pad1) -> Net-(J21-Pad4)
- MX2 pad 2: Net-(J22-Pad1) -> Net-(J15-Pad1)
- MX3 pad 1: Net-(J20-Pad1) -> Net-(J21-Pad4)
- MX4 pad 1: Net-(J20-Pad1) -> Net-(J21-Pad4)
- MX4 pad 2: Net-(J21-Pad2) -> Net-(J44-Pad2)
- MX5 pad 1: Net-(J20-Pad1) -> Net-(J21-Pad4)
- MX5 pad 2: Net-(J22-Pad2) -> Net-(J15-Pad2)
- MX6 pad 1: Net-(J20-Pad1) -> Net-(J21-Pad4)
- MX7 pad 1: Net-(J20-Pad1) -> Net-(J21-Pad4)
- MX7 pad 2: Net-(J21-Pad3) -> Net-(J44-Pad3)
- MX8 pad 1: Net-(J20-Pad1) -> Net-(J21-Pad4)
- MX8 pad 2: Net-(J22-Pad3) -> Net-(J15-Pad3)
- MX9 pad 1: Net-(J20-Pad1) -> Net-(J21-Pad4)
Routing:
- net Net-(J20-Pad1): track 291.0 -> 0.00 mm
- net Net-(J21-Pad4): track 8.90 -> 265.2 mm
- net Net-(J44-Pad1): track 0.00 -> 134.7 mm
- net Net-(J15-Pad1): track 0.00 -> 133.5 mm
- net Net-(J15-Pad2): track 0.00 -> 106.2 mm
- net Net-(J44-Pad2): track 0.00 -> 104.7 mm
- net Net-(J15-Pad3): track 0.00 -> 91.8 mm
- net Net-(J44-Pad3): track 0.00 -> 86.1 mm
- net Net-(J21-Pad1): track 84.3 -> 0.00 mm
- net Net-(J22-Pad1): track 84.2 -> 1.10 mm
- net Net-(J15-Pad4): track 0.00 -> 82.1 mm
- net Net-(J44-Pad4): track 0.00 -> 72.2 mm
- net Net-(J21-Pad2): track 52.9 -> 0.00 mm
- net Net-(J22-Pad2): track 53.3 -> 0.55 mm
- net Net-(J22-Pad3): track 31.3 -> 0.00 mm
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
Commit message: Tracing the plates.
Parts:
- added R4: 5.1K, Resistor_SMD:R_0402_1005Metric, B.Cu at (111.0, 466.4)
- added R5: 5.1K, Resistor_SMD:R_0402_1005Metric, B.Cu at (172.1, 467.1)
- C1, C10, C11, C12, C13, C14, C15, C16, C17, C18, C19, C2, C20, C21, C22, C23, C24, C25, C26, C27, C28, C29, C3, C30, C31, C32, C4, C5, C6, C7, C8, C9: footprint Capacitor_SMD:C_0805_2012Metric -> Capacitor_SMD:C_0402_1005Metric
- R10, R11, R12, R13, R14, R15, R16, R3, R6, R7, R8, R9: footprint Resistor_SMD:R_0805_2012Metric -> Resistor_SMD:R_0402_1005Metric
- moved R11 157.6 mm to (161.5, 392.6)
- moved R10 128.8 mm to (161.5, 393.7), turned to 180 degrees
- moved R8 126.7 mm to (123.3, 392.7)
- moved R9 125.1 mm to (123.3, 393.8), turned to 180 degrees
- moved F1 119.6 mm to (110.8, 407.0), turned to 180 degrees
- moved U2 114.1 mm to (165.0, 443.0), turned to 270 degrees
- moved F2 100.7 mm to (172.9, 400.9), turned to 90 degrees
- moved IC4 100.4 mm to (162.5, 462.2), turned to 270 degrees
- moved R2 95.6 mm to (119.2, 440.4), turned to 90 degrees
- moved R1 92.5 mm to (117.1, 440.3), turned to 90 degrees
- moved C18 76.4 mm to (220.0, 506.9)
- moved C26 75.9 mm to (220.2, 502.9)
- moved BOOTSEL2 75.4 mm to (207.2, 460.0), turned to 195 degrees
- moved C25 75.3 mm to (217.3, 499.6)
- moved C19 75.2 mm to (214.4, 501.6)
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Connections:
- C1 pad 1: L-RING1 -> +3V3
- C10 pad 1: L-RING1 -> +3V3
- C11 pad 1: L-RING1 -> +3V3
- C15 pad 1: L-RING1 -> +3V3
- C16 pad 1: L-RING1 -> +3V3
- C17 pad 1: L-RING1 -> +3V3
- C18 pad 1: L-RING1 -> +3V3
- C19 pad 1: L-RING1 -> +3V3
- C2 pad 1: L-RING1 -> +3V3
- C20 pad 1: L-RING1 -> +3V3
- C23 pad 1: L-RING1 -> +3V3
- C25 pad 1: L-RING1 -> +3V3
- C27 pad 1: L-RING1 -> +3V3
- C29 pad 1: L-RING1 -> +3V3
- C3 pad 1: L-RING1 -> +3V3
- C30 pad 1: L-RING1 -> +3V3
- C31 pad 1: L-RING1 -> +3V3
- C32 pad 1: L-RING1 -> +3V3
- C6 pad 1: L-RING1 -> +3V3
- C7 pad 1: L-RING1 -> +3V3
- C8 pad 1: +5V -> L-RING1
- C9 pad 1: +5V -> L-RING1
- F1 pad 1: +5V -> L-RING1
- F1 pad 2: Net-(F1-Pad2) -> +5VA
- F2 pad 1: +5V -> L-RING1
- F2 pad 2: Net-(F2-Pad2) -> +5VA
- IC1 pad 1: L-RING1 -> +3V3
- IC1 pad 10: L-RING1 -> +3V3
- IC1 pad 22: L-RING1 -> +3V3
- IC1 pad 3: ROW1 -> Net-(IC1-Pad3)
- IC1 pad 33: L-RING1 -> +3V3
- IC1 pad 34: COL4 -> Net-(IC1-Pad34)
- IC1 pad 35: COL0 -> Net-(IC1-Pad35)
- IC1 pad 36: COL1 -> Net-(IC1-Pad36)
- IC1 pad 37: COL2 -> Net-(IC1-Pad37)
- IC1 pad 38: COL3 -> Net-(IC1-Pad38)
- IC1 pad 39: COL5 -> Net-(IC1-Pad39)
- IC1 pad 4: COL7 -> Net-(IC1-Pad4)
- IC1 pad 40: ROW3 -> Net-(IC1-Pad40)
- IC1 pad 41: ROW2 -> Net-(IC1-Pad41)
- IC1 pad 42: L-RING1 -> +3V3
- IC1 pad 43: L-RING1 -> +3V3
- IC1 pad 44: L-RING1 -> +3V3
- IC1 pad 48: L-RING1 -> +3V3
- IC1 pad 49: L-RING1 -> +3V3
- IC1 pad 5: COL6 -> Net-(IC1-Pad5)
- IC1 pad 6: COL8 -> Net-(IC1-Pad6)
- IC1 pad 7: COL9 -> Net-(IC1-Pad7)
- IC1 pad 8: COLA -> Net-(IC1-Pad8)
- IC1 pad 9: COLB -> Net-(IC1-Pad9)
- IC2 pad 8: L-RING1 -> +3V3
- IC3 pad 1: L-RING1 -> +3V3
- IC3 pad 10: L-RING1 -> +3V3
- IC3 pad 22: L-RING1 -> +3V3
- IC3 pad 3: ROW1 -> Net-(IC3-Pad3)
- IC3 pad 33: L-RING1 -> +3V3
- IC3 pad 34: COL4 -> Net-(IC3-Pad34)
- IC3 pad 35: COL0 -> Net-(IC3-Pad35)
- IC3 pad 36: COL1 -> Net-(IC3-Pad36)
- IC3 pad 37: COL2 -> Net-(IC3-Pad37)
- IC3 pad 38: COL3 -> Net-(IC3-Pad38)
- IC3 pad 39: COL5 -> Net-(IC3-Pad39)
- IC3 pad 4: COL7 -> Net-(IC3-Pad4)
- IC3 pad 40: ROW3 -> Net-(IC3-Pad40)
- IC3 pad 41: ROW2 -> Net-(IC3-Pad41)
- IC3 pad 42: L-RING1 -> +3V3
- IC3 pad 43: L-RING1 -> +3V3
- IC3 pad 44: L-RING1 -> +3V3
- IC3 pad 48: L-RING1 -> +3V3
- IC3 pad 49: L-RING1 -> +3V3
- IC3 pad 5: COL6 -> Net-(IC3-Pad5)
- IC3 pad 6: COL8 -> Net-(IC3-Pad6)
- IC3 pad 7: COL9 -> Net-(IC3-Pad7)
- IC3 pad 8: COLA -> Net-(IC3-Pad8)
- IC3 pad 9: COLB -> Net-(IC3-Pad9)
- IC4 pad 8: L-RING1 -> +3V3
- J12 pad 1: Net-(J12-Pad1) -> K_K
- J12 pad 2: Net-(J12-Pad2) -> K_L
- J12 pad 3: Net-(J12-Pad3) -> K_SEMICOL
- J12 pad 4: Net-(J12-Pad4) -> K_ENT
- J19 pad 4: Net-(J19-Pad4) -> L-BASE
- J24 pad 1: L-BASE -> Net-(J24-Pad1)
- J25 pad 1: K_BSPC -> Net-(J25-Pad1)
- J25 pad 2: K_P -> Net-(J25-Pad2)
- J25 pad 3: K_O -> Net-(J25-Pad3)
- J25 pad 4: K_I -> L-BASE
- J26 pad 1: K_K -> Net-(J26-Pad1)
- J26 pad 2: K_L -> Net-(J26-Pad2)
- J26 pad 3: K_SEMICOL -> Net-(J26-Pad3)
- J26 pad 4: K_ENT -> Net-(J26-Pad4)
- J32 pad A4: Net-(F1-Pad2) -> +5VA
- J32 pad A9: Net-(F1-Pad2) -> +5VA
- J32 pad B4: Net-(F1-Pad2) -> +5VA
- J32 pad B9: Net-(F1-Pad2) -> +5VA
- J37 pad A4: Net-(F2-Pad2) -> +5VA
- J37 pad A9: Net-(F2-Pad2) -> +5VA
- J37 pad B4: Net-(F2-Pad2) -> +5VA
- J37 pad B9: Net-(F2-Pad2) -> +5VA
- J43 pad 1: Net-(J43-Pad1) -> K_BSPC
- J43 pad 2: Net-(J43-Pad2) -> K_P
- J43 pad 3: Net-(J43-Pad3) -> K_O
- J43 pad 4: Net-(J43-Pad4) -> K_I
- J9 pad 4: Net-(J9-Pad4) -> L-BASE
- MX31 pad 1: Net-(J28-Pad1) -> Net-(J29-Pad4)
- MX31 pad 2: Net-(J29-Pad4) -> Net-(J42-Pad4)
- MX32 pad 1: Net-(J28-Pad1) -> Net-(J29-Pad4)
- MX32 pad 2: Net-(J30-Pad1) -> Net-(J11-Pad1)
- MX33 pad 1: Net-(J28-Pad1) -> Net-(J29-Pad4)
- MX35 pad 1: Net-(J28-Pad1) -> Net-(J29-Pad4)
- MX35 pad 2: Net-(J29-Pad3) -> Net-(J42-Pad3)
- MX36 pad 1: Net-(J28-Pad1) -> Net-(J29-Pad4)
- MX36 pad 2: Net-(J30-Pad2) -> Net-(J11-Pad2)
- MX37 pad 1: Net-(J28-Pad1) -> Net-(J29-Pad4)
- MX39 pad 1: Net-(J28-Pad1) -> Net-(J29-Pad4)
- MX39 pad 2: Net-(J29-Pad2) -> Net-(J42-Pad2)
- MX40 pad 1: Net-(J28-Pad1) -> Net-(J29-Pad4)
- MX40 pad 2: Net-(J30-Pad3) -> Net-(J11-Pad3)
- MX41 pad 1: Net-(J28-Pad1) -> Net-(J29-Pad4)
- MX42 pad 1: Net-(J28-Pad1) -> Net-(J29-Pad4)
- MX42 pad 2: Net-(J29-Pad1) -> Net-(J42-Pad1)
- MX43 pad 1: Net-(J28-Pad1) -> Net-(J29-Pad4)
- MX43 pad 2: Net-(J30-Pad4) -> Net-(J11-Pad4)
- MX44 pad 1: Net-(J28-Pad1) -> Net-(J29-Pad4)
- R13 pad 2: L-RING1 -> +3V3
- R7 pad 2: L-RING1 -> +3V3
- U1 pad 2: L-RING1 -> +3V3
- U1 pad 3: +5V -> L-RING1
- U2 pad 2: L-RING1 -> +3V3
- U2 pad 3: +5V -> L-RING1
Routing:
- net L-BASE: track 0.00 -> 501.2 mm
- net Net-(J28-Pad1): track 323.3 -> 0.00 mm
- net Net-(J29-Pad4): track 8.57 -> 324.9 mm
- net Net-(J11-Pad4): track 0.00 -> 126.9 mm
- net Net-(J42-Pad1): track 0.00 -> 126.6 mm
- net L-RING1: track 0.00 -> 106.3 mm
- net Net-(J11-Pad3): track 0.00 -> 102.7 mm
- net Net-(J42-Pad2): track 0.00 -> 98.4 mm
- net Net-(J11-Pad2): track 0.00 -> 88.3 mm
- net Net-(J29-Pad1): track 85.0 -> 0.00 mm
- net Net-(J30-Pad4): track 83.7 -> 0.00 mm
- net Net-(J42-Pad3): track 0.00 -> 79.7 mm
- net Net-(J11-Pad1): track 0.00 -> 73.8 mm
- net Net-(J42-Pad4): track 0.00 -> 64.6 mm
- net Net-(J29-Pad2): track 55.4 -> 0.00 mm
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Other:
- net class Power added: clearance 0.2, trace_width 0.5, via_dia 0.8, via_drill 0.4
