File: ThumbsUp.kicad_pcb (KiCad board)
At the start: 2 copper layers, 247.3 x 260.9 mm, 152 parts, among them IC1 RP2040, IC2 W25Q128JVSIM, IC3 RP2040, IC4 W25Q128JVSIM, J1 Conn_01x04_Male, J10 Raiser_Male, J11 Raiser_Female, J12 Raiser_Male, J13 Raiser_Female, J14 Raiser_Male, J15 Raiser_Female, J16 Raiser_Male, J17 Raiser_Female, J18 Raiser_Male, J19 Raiser_Female, J2 Conn_01x04_Male, J20 Conn_01x04_Female, J21 Conn_01x04_Female, J22 Conn_01x04_Female, J23 Conn_01x04_Female, J24 Conn_01x04_Male, J25 Conn_01x04_Male, J26 Conn_01x04_Male, J27 Conn_01x04_Male, J28 Conn_01x04_Female, J29 Conn_01x04_Female, J3 Conn_01x04_Female, J30 Conn_01x04_Female, J31 Conn_01x04_Female, J32 USB_C_Receptacle_USB2.0, J33 Raiser_Male, J34 Raiser_Female, J35 Raiser_Male, J36 STX-3501-3N, J37 USB_C_Receptacle_USB2.0, J38 Raiser_Female, J39 Raiser_Male, J4 Conn_01x04_Male, J40 Raiser_Female, J41 Raiser_Male, J42 Raiser_Female, J43 Raiser_Male, J44 Raiser_Female, J45 Raiser_Male, J46 STX-3501-3N, J47 Raiser_Female, J48 Raiser_Male, J5 Conn_01x04_Female, J6 Conn_01x04_Male, J7 Conn_01x04_Male, J8 Conn_01x04_Male, J9 Raiser_Female, U1 NCP1117-3.3_SOT223, U2 NCP1117-3.3_SOT223, Y1 ABLS-12.000MHZ-B4-T, Y2 ABLS-12.000MHZ-B4-T

Commit message: Added mounting holes, silkscreens
Parts:
- added G***: LOGO, Silkscreens:Crowfeet75, B.Cu at (141.0, 584.0)
- added G***: LOGO, Silkscreens:Crowfeet75, F.Cu at (141.0, 566.0)
- added G***: LOGO, Silkscreens:Crowfeet75, F.Cu at (141.0, 410.0)
Routing:
- net Net-(J23-Pad3): track 29.0 -> 65.8 mm
- net Net-(J31-Pad2): track 31.5 -> 59.9 mm
- net Net-(J23-Pad2): track 53.3 -> 78.2 mm
- net Net-(J31-Pad3): track 54.5 -> 72.6 mm
- net Net-(J23-Pad1): track 85.0 -> 102.6 mm
- net Net-(J31-Pad4): track 83.4 -> 95.0 mm
- net Net-(J11-Pad4): track 126.9 -> 138.0 mm
- net Net-(J11-Pad3): track 102.7 -> 113.6 mm
- net Net-(J11-Pad2): track 88.3 -> 97.6 mm
- net Net-(J15-Pad1): track 131.9 -> 140.8 mm
- net Net-(J15-Pad2): track 106.2 -> 115.0 mm
- net Net-(J15-Pad3): track 91.8 -> 97.1 mm
- net Net-(J15-Pad4): track 82.1 -> 85.0 mm
- net Net-(J31-Pad1): track 8.34 -> 8.95 mm
Other:
- outline, holes or cut-outs redrawn

Commit message: Fixed the missing connectors and handiness pins
Parts:
- removed the G*** at (141.0, 584.0)
- removed the G*** at (141.0, 566.0)
- removed the G*** at (141.0, 410.0)
- added G***: LOGO, Silkscreens:Crowfeet75, B.Cu at (140.7, 560.2)
- added G***: LOGO, Silkscreens:Crowfeet75, F.Cu at (138.7, 559.7)
- added G***: LOGO, Silkscreens:Crowfeet75, F.Cu at (141.1, 403.8)
- added R17: 5.1K, Resistor_SMD:R_0402_1005Metric, B.Cu at (118.9, 466.8)
- R4, R5: value DNF -> 5.1K; footprint Resistor_SMD:R_0805_2012Metric -> Resistor_SMD:R_0402_1005Metric
- moved Y2 2.50 mm to (186.7, 456.6)
- moved C16 1.05 mm to (114.4, 455.4)
- moved R5 0.65 mm to (160.6, 444.9)
- moved R4 0.42 mm to (118.9, 468.3)
Connections:
- IC1 pad 4: Net-(IC1-Pad4) -> K_V
- IC1 pad 5: Net-(IC1-Pad5) -> K_LCTL
- IC1 pad 6: Net-(IC1-Pad6) -> K_Z
- IC1 pad 7: Net-(IC1-Pad7) -> K_X
- IC1 pad 8: K_V -> K_C
- IC3 pad 15: Net-(IC3-Pad15) -> K_RCTL
- IC3 pad 16: Net-(IC3-Pad16) -> K_SLASH
- IC3 pad 17: Net-(IC3-Pad17) -> K_DOT
- IC3 pad 18: Net-(IC3-Pad18) -> K_COMM
- IC3 pad 29: Net-(IC3-Pad29) -> L-BASE
Routing:
- net K_C: track 0.00 -> 46.9 mm
- net L-BASE: track 781.1 -> 827.5 mm, vias 26 -> 30
- net K_X: track 0.00 -> 43.6 mm
- net K_Z: track 0.00 -> 40.3 mm
- net K_LCTL: track 0.00 -> 35.7 mm
- net K_RCTL: track 0.00 -> 34.3 mm
- net K_SLASH: track 0.00 -> 33.9 mm
- net K_DOT: track 0.00 -> 33.6 mm
- net K_COMM: track 0.00 -> 33.3 mm
- net +3V3: track 215.0 -> 222.4 mm, vias 17 -> 18
- net Net-(IC3-Pad26): track 33.9 -> 27.1 mm, vias 4 -> 3
- net K_BSPC: track 44.5 -> 39.4 mm, vias 2 -> 1
- net Net-(IC1-Pad29): track 0.00 -> 4.07 mm
- net K_RALT: track 28.0 -> 31.3 mm
- net K_MNU: track 42.8 -> 46.2 mm
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